Commit message: Mesh file package name fix.

File: kubot_description/urdf/ur5.urdf.xacro (robot description, xacro)
@@ -72,13 +72,13 @@
       <visual>
         <geometry>
-          <mesh filename="package://ur_description/meshes/ur5/visual/base.dae" />
-        </geometry>
-        <material name="LightGrey">
-          <color rgba="0.7 0.7 0.7 1.0"/>
-        </material>
-      </visual>
-      <collision>
-        <geometry>
-          <mesh filename="package://ur_description/meshes/ur5/collision/base.stl" />
+          <mesh filename="package://kubot_description/meshes/ur5/visual/base.dae" />
+        </geometry>
+        <material name="LightGrey">
+          <color rgba="0.7 0.7 0.7 1.0"/>
+        </material>
+      </visual>
+      <collision>
+        <geometry>
+          <mesh filename="package://kubot_description/meshes/ur5/collision/base.stl" />
         </geometry>
       </collision>
@@ -103,13 +103,13 @@
       <visual>
         <geometry>
-          <mesh filename="package://ur_description/meshes/ur5/visual/shoulder.dae" />
-        </geometry>
-        <material name="LightGrey">
-          <color rgba="0.7 0.7 0.7 1.0"/>
-        </material>
-      </visual>
-      <collision>
-        <geometry>
-          <mesh filename="package://ur_description/meshes/ur5/collision/shoulder.stl" />
+          <mesh filename="package://kubot_description/meshes/ur5/visual/shoulder.dae" />
+        </geometry>
+        <material name="LightGrey">
+          <color rgba="0.7 0.7 0.7 1.0"/>
+        </material>
+      </visual>
+      <collision>
+        <geometry>
+          <mesh filename="package://kubot_description/meshes/ur5/collision/shoulder.stl" />
         </geometry>
       </collision>
@@ -134,13 +134,13 @@
       <visual>
         <geometry>
-          <mesh filename="package://ur_description/meshes/ur5/visual/upperarm.dae" />
-        </geometry>
-        <material name="LightGrey">
-          <color rgba="0.7 0.7 0.7 1.0"/>
-        </material>
-      </visual>
-      <collision>
-        <geometry>
-          <mesh filename="package://ur_description/meshes/ur5/collision/upperarm.stl" />
+          <mesh filename="package://kubot_description/meshes/ur5/visual/upperarm.dae" />
+        </geometry>
+        <material name="LightGrey">
+          <color rgba="0.7 0.7 0.7 1.0"/>
+        </material>
+      </visual>
+      <collision>
+        <geometry>
+          <mesh filename="package://kubot_description/meshes/ur5/collision/upperarm.stl" />
         </geometry>
       </collision>
@@ -165,13 +165,13 @@
       <visual>
         <geometry>
-          <mesh filename="package://ur_description/meshes/ur5/visual/forearm.dae" />
-        </geometry>
-        <material name="LightGrey">
-          <color rgba="0.7 0.7 0.7 1.0"/>
-        </material>
-      </visual>
-      <collision>
-        <geometry>
-          <mesh filename="package://ur_description/meshes/ur5/collision/forearm.stl" />
+          <mesh filename="package://kubot_description/meshes/ur5/visual/forearm.dae" />
+        </geometry>
+        <material name="LightGrey">
+          <color rgba="0.7 0.7 0.7 1.0"/>
+        </material>
+      </visual>
+      <collision>
+        <geometry>
+          <mesh filename="package://kubot_description/meshes/ur5/collision/forearm.stl" />
         </geometry>
       </collision>
@@ -196,13 +196,13 @@
       <visual>
         <geometry>
-          <mesh filename="package://ur_description/meshes/ur5/visual/wrist1.dae" />
-        </geometry>
-        <material name="LightGrey">
-          <color rgba="0.7 0.7 0.7 1.0"/>
-        </material>
-      </visual>
-      <collision>
-        <geometry>
-          <mesh filename="package://ur_description/meshes/ur5/collision/wrist1.stl" />
+          <mesh filename="package://kubot_description/meshes/ur5/visual/wrist1.dae" />
+        </geometry>
+        <material name="LightGrey">
+          <color rgba="0.7 0.7 0.7 1.0"/>
+        </material>
+      </visual>
+      <collision>
+        <geometry>
+          <mesh filename="package://kubot_description/meshes/ur5/collision/wrist1.stl" />
         </geometry>
       </collision>
@@ -227,13 +227,13 @@
       <visual>
         <geometry>
-          <mesh filename="package://ur_description/meshes/ur5/visual/wrist2.dae" />
-        </geometry>
-        <material name="LightGrey">
-          <color rgba="0.7 0.7 0.7 1.0"/>
-        </material>
-      </visual>
-      <collision>
-        <geometry>
-          <mesh filename="package://ur_description/meshes/ur5/collision/wrist2.stl" />
+          <mesh filename="package://kubot_description/meshes/ur5/visual/wrist2.dae" />
+        </geometry>
+        <material name="LightGrey">
+          <color rgba="0.7 0.7 0.7 1.0"/>
+        </material>
+      </visual>
+      <collision>
+        <geometry>
+          <mesh filename="package://kubot_description/meshes/ur5/collision/wrist2.stl" />
         </geometry>
       </collision>
@@ -258,13 +258,13 @@
       <visual>
         <geometry>
-          <mesh filename="package://ur_description/meshes/ur5/visual/wrist3.dae" />
-        </geometry>
-        <material name="LightGrey">
-          <color rgba="0.7 0.7 0.7 1.0"/>
-        </material>
-      </visual>
-      <collision>
-        <geometry>
-          <mesh filename="package://ur_description/meshes/ur5/collision/wrist3.stl" />
+          <mesh filename="package://kubot_description/meshes/ur5/visual/wrist3.dae" />
+        </geometry>
+        <material name="LightGrey">
+          <color rgba="0.7 0.7 0.7 1.0"/>
+        </material>
+      </visual>
+      <collision>
+        <geometry>
+          <mesh filename="package://kubot_description/meshes/ur5/collision/wrist3.stl" />
         </geometry>
       </collision>
