Commit message: Table added.

File: kubot_description/urdf/kubot_description.urdf.xacro (robot description, xacro)
@@ -10,9 +10,15 @@
     <xacro:ur5_robot prefix="arm_" joint_limited="false"/>
     <link name="world" />
-    <joint name="world_joint" type="fixed">
-      <parent link="world" />
-      <child link = "arm_base_link" />
-      <origin xyz="0.0 0.0 0.0" rpy="0.0 0.0 0.0" />
+    <xacro:include filename="$(find kubot_description)/urdf/table.xacro" />
+	   <joint name="world_joint" type="fixed">
+		   <origin xyz="0.40488474042 0.27988474042 0.3" rpy="0 0 0" />
+		     <parent link="world"/>
+		     <child link="table_base"/>
     </joint>
+	   <joint name="table_to_arm" type="fixed">
+		   <origin xyz="0 0 0" rpy="0 0 3.14159265359" />
+		     <parent link="tabletop_corner"/>
+		     <child link="arm_base_link"/>
+     </joint>
     <xacro:property name="M_PI" value="3.14159"/>
     <xacro:bhand_macro name="hand" parent="arm_ee_link">

Commit message: Kinect added.

File: kubot_description/urdf/kubot_description.urdf.xacro (robot description, xacro)
@@ -1,4 +1,5 @@
 <?xml version="1.0"?>
 <robot name="kubot" xmlns:xacro="http://ros.org/wiki/xacro">
+    <xacro:property name="M_PI" value="3.14159"/>
     <!-- Included URDF/XACRO Files -->
     <xacro:include filename="$(find kubot_description)/urdf/bh280.urdf.xacro" />
@@ -9,19 +10,22 @@
     <!-- arm -->
     <xacro:ur5_robot prefix="arm_" joint_limited="false"/>
+    <!-- kinect -->
+    <xacro:include filename="$(find kubot_description)/urdf/sensors/kinect.urdf.xacro"/>
     <link name="world" />
+    <!-- table -->
     <xacro:include filename="$(find kubot_description)/urdf/table.xacro" />
 	   <joint name="world_joint" type="fixed">
-		   <origin xyz="0.40488474042 0.27988474042 0.3" rpy="0 0 0" />
+		   <origin xyz="0 0 0.3" rpy="0 0 0" />
 		     <parent link="world"/>
 		     <child link="table_base"/>
     </joint>
 	   <joint name="table_to_arm" type="fixed">
-		   <origin xyz="0 0 0" rpy="0 0 3.14159265359" />
+		   <origin xyz="0 0 0" rpy="0 0 ${M_PI}" />
 		     <parent link="tabletop_corner"/>
 		     <child link="arm_base_link"/>
      </joint>
-    <xacro:property name="M_PI" value="3.14159"/>
     <xacro:bhand_macro name="hand" parent="arm_ee_link">
         <origin xyz="0 0 0" rpy="${M_PI/2} 0 ${M_PI/2}"/>
     </xacro:bhand_macro>
+    <sensor_kinect  parent="tabletop_other_corner"/>
 </robot>

File: kubot_description/urdf/table.xacro (robot description, xacro)
@@ -115,3 +115,9 @@
         <child link="tabletop_corner"/>
     </joint>
+    <link name="tabletop_other_corner"/>
+    <joint name="set_tabletop_relto__other_corner" type="fixed">
+        <origin xyz="-0.62 -0.44 0" rpy="0 0 -0.76" /> <!-- exact 45 degrees of -0.785398163397458 does not match the real table -->
+        <parent link="tabletop_ontop"/>
+        <child link="tabletop_other_corner"/>
+    </joint>
 </root>
