Commit message: Much better positions and simulation environment.

File: kubot_description/urdf/kinect_gazebo.urdf.xacro (robot description, xacro)
@@ -15,5 +15,5 @@
           <clip>
             <near>0.01</near>
-            <far>1.1</far>
+            <far>1.2</far>
           </clip>
         </camera>

File: kubot_description/urdf/kinect_properties.urdf.xacro (robot description, xacro)
@@ -19,9 +19,9 @@
      (currently in development and awaiting feedback)
    -->
-	<xacro:property name="cam_px" value="0" />
-  <xacro:property name="cam_py" value="0" />
+	<xacro:property name="cam_px" value="-0.1" />
+  <xacro:property name="cam_py" value="-0.1" />
 	<xacro:property name="cam_pz" value="0.5" />
 	<xacro:property name="cam_or" value="0" />
 	<xacro:property name="cam_op" value="${M_PI/4}" />
-	<xacro:property name="cam_oy" value="${M_PI/2}" />
+	<xacro:property name="cam_oy" value="${2.2*M_PI/5}" />
 </robot>

File: kubot_gazebo/objects/basic_cube.urdf (robot description, URDF)
Before this commit: robot basic_box, 1 links, 0 joints
Links:
- link box_link: geometry collision box size=0.1 0.1 0.1; visual box size=0.1 0.1 0.1

File: kubot_gazebo/objects/basic_sphere.urdf (robot description, URDF)
Before this commit: robot basic_sphere, 1 links, 0 joints
Links:
- link sphere_link: mass 0.01 -> 0.001; geometry collision sphere radius=0.05; visual sphere radius=0.05
