Commit message: Started dataset collection

File: kubot_gazebo/objects/basic_cube.urdf (robot description, URDF)
Before this commit: robot basic_box, 1 links, 0 joints
Links:
- removed link base_link
- added link box_link, mass 0.01; collision box size=0.15 0.15 0.15; visual box size=0.15 0.15 0.15
